File: XX-Piezo-Reciever.brd (EAGLE design)
At the start: 160 x 100 mm, 9 parts, among them IC1 TL072D, IC2 TL072D, J1 AVR_SPI_PROG_3X2PTH, U1 ATMEGA1284P-AU

Commit message: Finished routing, first complete version
Parts:
- R3, R4: device resistor:R01005 -> rcl:R0402
- moved IC2 51.6 mm to (66.5, 44.7), turned to 270 degrees
- moved R4 45.8 mm to (59.7, 45.2), turned to 90 degrees
- moved R2 39.0 mm to (59.7, 41.4), turned to 90 degrees
- moved IC1 31.3 mm to (66.5, 37.8), turned to 270 degrees
- moved R1 28.0 mm to (59.7, 34.0), turned to 90 degrees
- moved R3 28.0 mm to (59.7, 37.8), turned to 90 degrees
- moved J2 1.27 mm to (70.1, 30.5)
Connections:
- removed net AVCC: U1.27
- net GND: now also U1.18, U1.28, U1.6
- net VCC: now also U1.27
Routing:
- net PIEZO-: track 0.00 -> 28.5 mm
- net PIEZO+: track 0.00 -> 22.4 mm
- net V+: track 0.00 -> 20.9 mm
- net OUT2: track 0.00 -> 16.4 mm
- net V-: track 0.00 -> 15.0 mm
- net VCC: track 13.4 -> 22.4 mm
- net PIEZO+1: track 0.00 -> 8.08 mm
- net PIEZO+2: track 0.00 -> 7.09 mm
- net OUT1: track 0.00 -> 6.95 mm
- net A1: track 18.6 -> 24.3 mm, vias 0 -> 1
- net GND: track 0.00 -> 5.33 mm, vias 0 -> 1
- added copper zone on layer 1, net GND
Other:
- outline, holes or cut-outs redrawn
- board text added: "5V"
- board text added: "A1"
- board text added: "Charles Li Joshua Burdine"
- board text added: "GND"
- board text added: "MISO"
- board text added: "MOSI"
- board text added: "PIEZO+"
- board text added: "PIEZO-"
- board text added: "R1"
- board text added: "R2"
- board text added: "R3"
- board text added: "R4"
- board text added: "RESET"
- board text added: "SCK"
- board text added: "V+"
- board text added: "V-"
