File: XX-Piezo-Reciever.sch (EAGLE design)
At the start: 9 parts, among them IC1 TL072D, IC2 TL072D, J1 AVR_SPI_PROG_3X2PTH, U1 ATMEGA1284P-AU

Commit message: Finished routing, first complete version
Parts:
- R3, R4: device resistor:R-US_01005 -> rcl:R-US_R0402
Connections:
- net GND: now also U1.GND_2, U1.GND_3, U1.GND_4
- net VCC: now also U1.AVCC
