File: XX-Piezo-Reciever.sch (EAGLE design)
At the start: 9 parts, among them IC1 TL072D, J1 AVR_SPI_PROG_3X2PTH, U1 ATMEGA1284P-AU

Commit message: Added correct mosfet, finished routing. No decoup caps yet.
Parts:
- removed Q1: (no value), m-pad-2.1:MOSFET_N_SOT223
- added IC2: L78LXXBD/CD, v-reg-3:L78LXXBD/CD
- added T1: (no value), zetex:NMOSSOT23
Connections:
- net +5V: now also IC2.OUT
- net +6V: now also IC2.IN
- net A1: now also T1.G; no longer Q1.G
- net GND: now also IC2.GND1, T1.S; no longer Q1.S
- net OUTPUT: now also T1.D; no longer Q1.D
Changed lines of the file:
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@@
 <?xml version="1.0" encoding="utf-8"?>
 <!DOCTYPE eagle SYSTEM "eagle.dtd">
-<eagle version="8.7.0">
+<eagle version="8.3.2">
 <drawing>
 <settings>
@@
 <setting verticaltext="up"/>
 </settings>
-<grid distance="50" unitdist="mil" unit="mil" style="dots" multiple="1" display="yes" altdistance="0.01" altunitdist="inch" altunit="inch"/>
+<grid distance="50" unitdist="mil" unit="mil" style="lines" multiple="1" display="yes" altdistance="0.01" altunitdist="inch" altunit="inch"/>
 <layers>
 <layer number="1" name="Top" color="4" fill="1" visible="no" active="no"/>
@@
 <part name="R4" library="rcl" library_urn="urn:adsk.eagle:library:334" deviceset="R-US_" device="R0402" package3d_urn="urn:adsk.eagle:package:23547/1" value="10k"/>
 <part name="GND3" library="supply1" library_urn="urn:adsk.eagle:library:371" deviceset="GND" device=""/>
-<part name="Q1" library="m-pad-2.1" deviceset="MOSFET_N_SOT223" device=""/>
 <part name="GND4" library="supply1" library_urn="urn:adsk.eagle:library:371" deviceset="GND" device=""/>
+<part name="IC2" library="v-reg-3" deviceset="L78LXXBD/CD" device=""/>
+<part name="GND5" library="supply1" library_urn="urn:adsk.eagle:library:371" deviceset="GND" device=""/>
+<part name="T1" library="zetex" library_urn="urn:adsk.eagle:library:418" deviceset="NMOSSOT23" device="" package3d_urn="urn:adsk.eagle:package:30981/1"/>
+<part name="+6V1" library="supply2" library_urn="urn:adsk.eagle:library:372" deviceset="V+" device="" value="+6V"/>
 </parts>
 <sheets>
@@
 <instance part="R4" gate="G$1" x="63.5" y="50.8"/>
 <instance part="GND3" gate="1" x="96.52" y="87.63"/>
-<instance part="Q1" gate="G$1" x="20.32" y="86.36" smashed="yes" rot="R180">
-<attribute name="NAME" x="25.4" y="82.55" size="1.778" layer="95" rot="R180"/>
-<attribute name="VALUE" x="15.24" y="86.36" size="1.778" layer="96" rot="R180"/>
-</instance>
 <instance part="GND4" gate="1" x="15.24" y="92.71"/>
+<instance part="IC2" gate="G$1" x="40.64" y="109.22"/>
+<instance part="GND5" gate="1" x="40.64" y="95.25"/>
+<instance part="T1" gate="A" x="20.32" y="86.36" rot="R180"/>
+<instance part="+6V1" gate="1" x="27.94" y="115.57"/>
 </instances>
 <busses>
@@
 <label x="90.17" y="97.79" size="1.778" layer="95"/>
 </segment>
+<segment>
+<pinref part="IC2" gate="G$1" pin="OUT"/>
+<wire x1="48.26" y1="109.22" x2="54.61" y2="109.22" width="0.1524" layer="91"/>
+<label x="49.53" y="109.22" size="1.778" layer="95"/>
+</segment>
 </net>
 <net name="MOSI" class="0">
@@
 <wire x1="-7.62" y1="81.28" x2="-17.78" y2="81.28" width="0.1524" layer="91"/>
 <wire x1="-17.78" y1="81.28" x2="-17.78" y2="85.09" width="0.1524" layer="91"/>
+</segment>
+<segment>
+<pinref part="IC2" gate="G$1" pin="IN"/>
+<wire x1="33.02" y1="109.22" x2="27.94" y2="109.22" width="0.1524" layer="91"/>
+<pinref part="+6V1" gate="1" pin="V+"/>
+<wire x1="27.94" y1="109.22" x2="27.94" y2="113.03" width="0.1524" layer="91"/>
 </segment>
 </net>
@@
 </segment>
 <segment>
-<pinref part="Q1" gate="G$1" pin="S"/>
 <wire x1="20.32" y1="91.44" x2="20.32" y2="96.52" width="0.1524" layer="91"/>
 <wire x1="20.32" y1="96.52" x2="15.24" y2="96.52" width="0.1524" layer="91"/>
 <pinref part="GND4" gate="1" pin="GND"/>
 <wire x1="15.24" y1="96.52" x2="15.24" y2="95.25" width="0.1524" layer="91"/>
+<pinref part="T1" gate="A" pin="S"/>
+</segment>
+<segment>
+<pinref part="IC2" gate="G$1" pin="GND1"/>
+<wire x1="40.64" y1="101.6" x2="40.64" y2="97.79" width="0.1524" layer="91"/>
+<pinref part="GND5" gate="1" pin="GND"/>
+<wire x1="40.64" y1="97.79" x2="40.64" y2="96.52" width="0.1524" layer="91"/>
 </segment>
 </net>
@@
 <segment>
 <pinref part="J2" gate="A" pin="4"/>
-<pinref part="Q1" gate="G$1" pin="D"/>
 <wire x1="0" y1="78.74" x2="20.32" y2="78.74" width="0.1524" layer="91"/>
 <wire x1="20.32" y1="78.74" x2="20.32" y2="81.28" width="0.1524" layer="91"/>
 <label x="10.16" y="78.74" size="1.778" layer="95"/>
+<pinref part="T1" gate="A" pin="D"/>
 </segment>
 </net>
 <net name="A1" class="0">
 <segment>
-<pinref part="Q1" gate="G$1" pin="G"/>
 <wire x1="25.4" y1="88.9" x2="30.48" y2="88.9" width="0.1524" layer="91"/>
 <label x="27.94" y="88.9" size="1.778" layer="95"/>
-</segment>
-<segment>
+<pinref part="T1" gate="A" pin="G"/>
+</segment>
+<segment>
